Commit message: adding in the second link to the arm

File: rrbot_description/urdf/rrbot.xacro (robot description, xacro)
@@ -76,4 +76,35 @@
     </inertial>
   </link>
+    <joint name="joint2" type="continuous">
+    <parent link="link2"/>
+    <child link="link3"/>
+    <origin xyz="0 ${width} ${height2 - axel_offset*2}" rpy="0 0 0"/>
+    <axis xyz="0 1 0"/>
+    <dynamics damping="0.7"/>
+  </joint>
+  <!-- Top Link -->
+  <link name="link3">
+    <collision>
+      <origin xyz="0 0 ${height3/2 - axel_offset}" rpy="0 0 0"/>
+      <geometry>
+	<box size="${width} ${width} ${height3}"/>
+      </geometry>
+    </collision>
+    <visual>
+      <origin xyz="0 0 ${height3/2 - axel_offset}" rpy="0 0 0"/>
+      <geometry>
+	<box size="${width} ${width} ${height3}"/>
+      </geometry>
+      <material name="blue"/>
+    </visual>
+    <inertial>
+      <origin xyz="0 0 ${height3/2 - axel_offset}" rpy="0 0 0"/>
+      <mass value="${mass}"/>
+      <inertia
+	  ixx="${mass / 12.0 * (width*width + height3*height3)}" ixy="0.0" ixz="0.0"
+	  iyy="${mass / 12.0 * (height3*height3 + width*width)}" iyz="0.0"
+	  izz="${mass / 12.0 * (width*width + width*width)}"/>
+    </inertial>
+  </link>
   <transmission name="tran1">
     <type>transmission_interface/SimpleTransmission</type>
@@ -86,3 +117,13 @@
     </actuator>
   </transmission>
+  <transmission name="tran2">
+    <type>transmission_interface/SimpleTransmission</type>
+    <joint name="joint2">
+      <hardwareInterface>hardware_interface/EffortJointInterface</hardwareInterface>
+    </joint>
+    <actuator name="motor2">
+      <hardwareInterface>hardware_interface/EffortJointInterface</hardwareInterface>
+      <mechanicalReduction>1</mechanicalReduction>
+    </actuator>
+  </transmission>
 </robot>

Commit message: adding max effort and velocity limits to arm joints

File: rrbot_description/urdf/rrbot.xacro (robot description, xacro)
@@ -9,4 +9,6 @@
   <xacro:property name="height2" value="1" /> <!-- Link 2 -->
   <xacro:property name="height3" value="1" /> <!-- Link 3 -->
+  <xacro:property name="max_effort" value="50" /> <!-- Max effort for joint -->
+  <xacro:property name="max_velocity" value="5" /> <!-- Max velocity for joint -->
   <xacro:property name="camera_link" value="0.05" /> <!-- Size of square 'camera' box -->
   <xacro:property name="axel_offset" value="0.05" /> <!-- Space btw top of beam and the each joint -->
@@ -51,4 +53,5 @@
     <axis xyz="0 1 0"/>
     <dynamics damping="0.7"/>
+    <limit effort="${max_effort}" velocity="${max_velocity}"/>
   </joint>
   <!-- Middle Link -->
@@ -76,5 +79,5 @@
     </inertial>
   </link>
-    <joint name="joint2" type="continuous">
+  <joint name="joint2" type="continuous">
     <parent link="link2"/>
     <child link="link3"/>
@@ -82,4 +85,5 @@
     <axis xyz="0 1 0"/>
     <dynamics damping="0.7"/>
+    <limit effort="${max_effort}" velocity="${max_velocity}"/>
   </joint>
   <!-- Top Link -->
